Commit message: Update

File: husky/husky_description/urdf/accessories/sick_lms1xx_mount.urdf.xacro (robot description, xacro)
@@ -50,4 +50,15 @@
       <child link="${prefix}_laser" />
     </joint>
+    <link name="laser">
+      <!--visual>
+        <origin xyz="0 0 0" rpy="0 0 0" />
+      </visual -->
+    </link>
+    <joint name="laser_connection" type="fixed">
+      <!-- This offset is from the base of the bracket to the LIDAR's focal point. -->
+      <origin xyz="0 0 0" rpy="0 0 0" />
+      <parent link="${prefix}_laser" />
+      <child link="laser" />
+    </joint>
   </xacro:macro>
 </robot>

File: husky/husky_description/urdf/decorations.urdf.xacro (robot description, xacro)
@@ -85,5 +85,5 @@
           <origin xyz="0 0 0" rpy="0 0 0" />
           <geometry>
-            <mesh filename="package://husky_description/meshes/top_plate.dae" />
+            <mesh filename="package://husky_description/meshes/top_plate.dae" scale="1.037 1 1"/>
           </geometry>
         </visual>
@@ -91,5 +91,5 @@
           <origin xyz="0 0 0" rpy="0 0 0"/>
           <geometry>
-            <mesh filename="package://husky_description/meshes/top_plate.stl" />
+            <mesh filename="package://husky_description/meshes/top_plate.stl" scale="1.037 1 1"/>
           </geometry>
         </collision>

File: husky/husky_description/urdf/description.xacro (robot description, xacro)
@@ -22,11 +22,12 @@
 -->
 <robot name="husky" xmlns:xacro="http://ros.org/wiki/xacro">
-  <xacro:arg name="laser_enabled" default="true" />
+  <xacro:arg name="laser_enabled" default="false" />
   <xacro:arg name="ur5_enabled" default="false" />
   <xacro:arg name="ur5_camera_enabled" default="false" />
   <xacro:arg name="ur5_mbzirc_gripper_enabled" default="true" />
   <xacro:arg name="kinect_enabled" default="false" />
-  <xacro:arg name="kinectv2_enabled" default="true" />
+  <xacro:arg name="kinectv2_enabled" default="false" />
   <xacro:arg name="primesense_enabled" default="false"/>
+  <xacro:arg name="velodyne_lidar" default="true"/>
   <xacro:include filename="$(find husky_description)/urdf/husky.urdf.xacro" />
   <xacro:husky_robot />

File: husky/husky_description/urdf/husky.urdf.xacro (robot description, xacro)
@@ -22,4 +22,12 @@
 -->
 <robot name="husky_robot" xmlns:xacro="http://ros.org/wiki/xacro">
+  <arg name="laser_enabled" default="false"/>
+  <arg name="ur5_enabled" default="true"/>
+  <arg name="ur5_camera_enabled" default="false"/>
+  <arg name="ur5_mbzirc_gripper_enabled" default="false" />
+  <arg name="kinect_enabled" default="false"/>
+  <arg name="kinectv2_enabled" default="false"/>
+  <arg name="primesense_enabled" default="false"/>
+  <arg name="velodyne_lidar" default="true"/>
   <!-- Included URDF/XACRO Files -->
   <xacro:include filename="$(find husky_description)/urdf/decorations.urdf.xacro" />
@@ -31,4 +39,6 @@
   <xacro:include filename="$(find husky_description)/urdf/accessories/sensor_arch.urdf.xacro"/>
   <xacro:include filename="$(find ur_description)/urdf/ur5.urdf.xacro" />
+  <xacro:include filename="$(find velodyne_description)/urdf/HDL-32E.urdf.xacro" />
+  <!-- xacro:include filename="$(find velodyne_description)/urdf/VLP-16.urdf.xacro" / -->
   <property name="M_PI" value="3.14159"/>
   <!-- Base Size -->
@@ -152,4 +162,19 @@
       </joint>
     </xacro:if>
+    <xacro:if value="$(arg velodyne_lidar)" >
+    <!--VLP-16 parent="top_plate_link" name="velodyne_link" topic="velodyne_points" >
+      <origin xyz="-0.35 0 0.51" rpy="0 0 0"/>
+    </VLP-16 -->
+    <HDL-32E parent="top_plate_link" name="velodyne_link" topic="velodyne_points" >
+        <origin xyz="0.44 0 -0.16" rpy="0 0 -1.57" />
+    </HDL-32E>
+      <!-- velodyne_vlp16_mount prefix="base" topic="velodyne_points"/ -->
+      <!-- joint name="laser_mount_joint" type="fixed">
+        <origin xyz="$(optenv HUSKY_LMS1XX_XYZ 0.415 0.0 -0.04)"
+                rpy="$(optenv HUSKY_LMS1XX_RPY 0.0 0.0 0.0)" />
+        <parent link="top_plate_link" />
+        <child link="base_laser_mount" />
+      </joint -->
+    </xacro:if>
     <!-- Spawn Kinect if kinect_enabled = "true" -->
     <xacro:if value="$(arg kinect_enabled)">

File: husky/husky_description/urdf/husky_ur5.urdf (robot description, URDF)
Before this commit: robot husky, 35 links, 34 joints
Joints:
- joint ur5_arm_wrist_1_joint: limit lower=-3.14159265 upper=3.14159265 effort=28.0 velocity=3.2 -> lower=-6.28 upper=6.28 effort=28.0 velocity=3.2

File: universal_robot/ur_description/urdf/ur5.urdf.xacro (robot description, xacro)
@@ -95,8 +95,9 @@
       <axis xyz="0 0 1" />
       <xacro:unless value="${joint_limited}">
-        <limit lower="${-2.0 * pi}" upper="${2.0 * pi}" effort="150.0" velocity="3.15"/>
-      </xacro:unless>
-      <xacro:if value="${joint_limited}">
-        <limit lower="${-pi}" upper="${pi}" effort="150.0" velocity="3.15"/>
+        <limit lower="0" upper="${0.75 * pi}" effort="150.0" velocity="3.15"/>
+        <!-- limit lower="${-2.0 * pi}" upper="0.25" effort="150.0" velocity="3.15"/ -->
+      </xacro:unless>
+      <xacro:if value="${joint_limited}">
+        <limit lower="0" upper="${0.75 * pi}" effort="150.0" velocity="3.15"/>
       </xacro:if>
       <dynamics damping="0.0" friction="0.0"/>
@@ -126,8 +127,8 @@
       <axis xyz="0 1 0" />
       <xacro:unless value="${joint_limited}">
-        <limit lower="${-2.0 * pi}" upper="${2.0 * pi}" effort="150.0" velocity="3.15"/>
-      </xacro:unless>
-      <xacro:if value="${joint_limited}">
-        <limit lower="${-pi}" upper="${pi}" effort="150.0" velocity="3.15"/>
+        <limit lower="${-1.0 * pi}" upper="${0.0 * pi}" effort="150.0" velocity="3.15"/>
+      </xacro:unless>
+      <xacro:if value="${joint_limited}">
+        <limit lower="${-1.0 * pi}" upper="${0.0 * pi}" effort="150.0" velocity="3.15"/>
       </xacro:if>
       <dynamics damping="0.0" friction="0.0"/>
@@ -157,8 +158,8 @@
       <axis xyz="0 1 0" />
       <xacro:unless value="${joint_limited}">
-        <limit lower="${-2.0 * pi}" upper="${2.0 * pi}" effort="150.0" velocity="3.15"/>
-      </xacro:unless>
-      <xacro:if value="${joint_limited}">
-        <limit lower="${-pi}" upper="${pi}" effort="150.0" velocity="3.15"/>
+        <limit lower="${0.0 * pi}" upper="${1.0 * pi}" effort="150.0" velocity="3.15"/>
+      </xacro:unless>
+      <xacro:if value="${joint_limited}">
+        <limit lower="${0.0 * pi}" upper="${1.0 * pi}" effort="150.0" velocity="3.15"/>
       </xacro:if>
       <dynamics damping="0.0" friction="0.0"/>
@@ -175,5 +176,7 @@
       <collision>
         <geometry>
-          <mesh filename="package://ur_description/meshes/ur5/collision/forearm.stl" />
+          <mesh filename="package://ur_description/meshes/ur5/collision/forearm.stl">
+            <scale>1.10 1.10 1.10</scale>
+          </mesh>
         </geometry>
       </collision>
@@ -188,8 +191,8 @@
       <axis xyz="0 1 0" />
       <xacro:unless value="${joint_limited}">
-        <limit lower="${-2.0 * pi}" upper="${2.0 * pi}" effort="28.0" velocity="3.2"/>
-      </xacro:unless>
-      <xacro:if value="${joint_limited}">
-        <limit lower="${-pi}" upper="${pi}" effort="28.0" velocity="3.2"/>
+        <limit lower="${0.5 * pi}" upper="${1.25 * pi}" effort="28.0" velocity="3.2"/>
+      </xacro:unless>
+      <xacro:if value="${joint_limited}">
+        <limit lower="${0.5 * pi}" upper="${1.25 * pi}" effort="28.0" velocity="3.2"/>
       </xacro:if>
       <dynamics damping="0.0" friction="0.0"/>
@@ -219,8 +222,8 @@
       <axis xyz="0 0 1" />
       <xacro:unless value="${joint_limited}">
-        <limit lower="${-2.0 * pi}" upper="${2.0 * pi}" effort="28.0" velocity="3.2"/>
-      </xacro:unless>
-      <xacro:if value="${joint_limited}">
-        <limit lower="${-pi}" upper="${pi}" effort="28.0" velocity="3.2"/>
+        <limit lower="${-1.0 * pi}" upper="${0.0 * pi}" effort="28.0" velocity="3.2"/>
+      </xacro:unless>
+      <xacro:if value="${joint_limited}">
+        <limit lower="${-1.0 * pi}" upper="${0.0 * pi}" effort="28.0" velocity="3.2"/>
       </xacro:if>
       <dynamics damping="0.0" friction="0.0"/>
@@ -253,5 +256,5 @@
       </xacro:unless>
       <xacro:if value="${joint_limited}">
-        <limit lower="${-pi}" upper="${pi}" effort="28.0" velocity="3.2"/>
+        <limit lower="${-2.0 * pi}" upper="${2.0 * pi}" effort="28.0" velocity="3.2"/>
       </xacro:if>
       <dynamics damping="0.0" friction="0.0"/>
